Commit message: Moved where the lidar is in the urdf

File: src/lumina/description/lidar.xacro (robot description, xacro)
@@ -4,5 +4,5 @@
         <parent link="chassis"/>
         <child link="laser_frame"/>
-        <origin xyz="0.12 0.0 0.22" rpy="0.0 0.0 0.0"/>
+        <origin xyz="0.20 0.0 0.22" rpy="0.0 0.0 0.0"/>
     </joint>
     <link name="laser_frame">
