Commit message: Added lidar xacro

File: src/lumina/description/robot.urdf.xacro (robot description, xacro)
@@ -3,3 +3,4 @@
     <xacro:include filename="robot_core.xacro" />
     <xacro:include filename="gazebo_control.xacro" />
+    <xacro:include filename="lidar.xacro" />
 </robot>

File: src/lumina/description/robot_core.xacro (robot description, xacro)
@@ -33,5 +33,5 @@
             <origin xyz="0.18 0.0 0.08" rpy="0.0 0.0 0.0" />
             <geometry>
-                <box size="0.24 0.24 0.16" />
+                <box size="0.24 0.24 0.18" />
             </geometry>
             <material name="white" />

Commit message: Working on updating to the ign version of gazebo since the classic version wasn't working well

File: src/lumina/description/robot.urdf.xacro (robot description, xacro)
@@ -1,7 +1,9 @@
 <?xml version="1.0"?>
-<robot xmlns:xacro="http://www.ros.org/wiki/xacro"  name="robot">
+<robot xmlns:xacro="http://www.ros.org/wiki/xacro" name="robot">
+    <xacro:include filename="inertial_macros.xacro"/>
     <xacro:include filename="robot_core.xacro" />
-    <xacro:include filename="gazebo_control.xacro" />
+    <!-- <xacro:include filename="gazebo_control.xacro" /> -->
     <xacro:include filename="lidar.xacro" />
     <xacro:include filename="camera.xacro" />
+    <xacro:include filename="ros2_control.xacro" />
 </robot>

File: src/lumina/description/robot_core.xacro (robot description, xacro)
@@ -1,8 +1,4 @@
 <?xml version="1.0"?>
-<robot xmlns:xacro="http://www.ros.org/wiki/xacro" name="lumina">
-    <xacro:include filename="inertial_macros.xacro"/>
-    <material name="white">
-        <color rgba="1 1 1 1" />
-    </material>
+<robot xmlns:xacro="http://www.ros.org/wiki/xacro">
     <material name="orange">
         <color rgba="1 0.3 0.1 1" />
@@ -16,4 +12,7 @@
     <material name="red">
         <color rgba="1 0 0 1" />
+    </material>
+    <material name="white">
+        <color rgba="1 1 1 1" />
     </material>
     <!-- BASE LINK -->

Commit message: Added imu xacro + mapper params

File: src/lumina/description/robot.urdf.xacro (robot description, xacro)
@@ -6,4 +6,5 @@
     <xacro:include filename="lidar.xacro" />
     <xacro:include filename="camera.xacro" />
+    <xacro:include filename="imu.xacro" />
     <xacro:include filename="ros2_control.xacro" />
 </robot>

File: src/lumina/description/robot_core.xacro (robot description, xacro)
@@ -19,4 +19,9 @@
     <link name="base_link">
     </link>
+    <joint name="base_footprint_joint" type="fixed">
+        <parent link="base_link" />
+        <child link="base_footprint" />
+        <origin xyz="0 0 0" rpy="0 0 0" />
+    </joint>
     <joint name="chassis_joint" type="fixed">
         <parent link="base_link" />
