Commit message: Got odom filtered working properly!

File: src/lumina/description/imu.xacro (robot description, xacro)
@@ -4,5 +4,5 @@
         <parent link="chassis"/>
         <child link="imu_frame" />
-        <origin xyz="0.0 0.0 0.8" rpy="0.0 0.0 0.0" />
+        <origin xyz="0.0 0.0 0.08" rpy="0.0 0.0 0.0" />
     </joint>
     <!-- IMU frame -->
@@ -19,5 +19,5 @@
             </geometry>
         </collision>
-        <xacro:inertial_box mass="0.05" size="0.05 0.05 0.02">
+        <xacro:inertial_box mass="0.05" x="0.05" y="0.05" z="0.02">
             <origin xyz="0.0 0.0 0.0" rpy="0.0 0.0 0.0"/>
         </xacro:inertial_box>

File: src/lumina/description/robot_core.xacro (robot description, xacro)
@@ -24,4 +24,6 @@
         <origin xyz="0 0 0" rpy="0 0 0" />
     </joint>
+    <link name="base_footprint">
+    </link>
     <joint name="chassis_joint" type="fixed">
         <parent link="base_link" />

File: src/lumina/description/ros2_control.xacro (robot description, xacro)
@@ -11,5 +11,5 @@
                 <param name="baud_rate">57600</param>
                 <param name="timeout">1000</param>
-                <param name="enc_counts_per_rev">341</param>
+                <param name="enc_counts_per_rev">1559</param>
             </hardware>
             <joint name="left_wheel_joint">
